File: KicadFiles/MacroBoard.kicad_pcb (KiCad board)
At the start: 2 copper layers, 94 x 116.1 mm, 79 parts, among them J1 USB_B_Micro, J2 Conn_01x08_Male, SW1 SW_Push, SW10 SW_Push, SW11 SW_Push, SW12 SW_Push, SW13 SW_Push, SW14 SW_Push, SW15 SW_Push, SW16 SW_Push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

Commit message: added logo
Parts:
- added G***: LOGO, Logo:logo, F.Cu at (78.4, 66.7)
Other:
- board text added: "Krzysztof Sikora Kacper Filipek"
- board text removed: "PCB by Kacper Filipek"
